File: MAR.kicad_sch (KiCad schematic)
At the start: 24 parts, among them J27 574_CP, J28 OE/A->B, Q25 BC557, Q26 BC547, Q27 BC547, U33 74HC574_w_Pwr, U36 74HC574_w_Pwr, U47 74HC245, U48 74HC245, U49 74HC245, U50 74HC245

Commit message: feat: added IR into motherboard
Parts:
- added C137: 100nF, Capacitor_THT:C_Disc_D3.0mm_W1.6mm_P2.50mm, symbol Device:C
- added U4: 74HC04, symbol 74xx:74HC04
Connections:
- net GND: now also C137.2, U4.7 (GND)
- net Vcc: now also C137.1, U4.14 (VCC)
- net MAR_ADDR_GATE#: no longer names the net of U47.19 (CE), U48.19 (CE)
- net MAR_ADDR_GATE#: now also U4.2
- net MAR_DATA_GATE# renamed MAR_GATE[0->DATA;1->ADDR]
- net MAR_GATE[0->DATA;1->ADDR]: now also U4.1
