File: IR.kicad_sch (KiCad schematic)
At the start: 20 parts, among them J42 574_CP, J43 OE/A->B, Q46 BC557, Q47 BC547, Q48 BC547, U133 74HC574_w_Pwr, U134 74HC245, U135 74HC245, U136 74HC574_w_Pwr

Commit message: WIP: created but not finished cl
Connections:
- net 0 renamed BIT0
- net RES0 renamed JCC0
- net RES1 renamed JCC1
- net RES2 renamed JCC2
Changed lines of the file:
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@@
 		)
 	)
-	(hierarchical_label "0"
+	(hierarchical_label "BIT0"
 		(shape output)
 		(at 128.27 30.48 90)
@@
 		)
 	)
-	(hierarchical_label "RES0"
+	(hierarchical_label "JCC0"
 		(shape output)
 		(at 125.73 30.48 90)
@@
 		)
 	)
+	(hierarchical_label "JCC1"
+		(shape output)
+		(at 123.19 30.48 90)
+		(effects
+			(font
+				(size 1.27 1.27)
+			)
+			(justify left)
+		)
+	)
 	(hierarchical_label "RS20"
 		(shape output)
@@
 		)
 	)
-	(hierarchical_label "RES1"
-		(shape output)
-		(at 123.19 30.48 90)
-		(effects
-			(font
-				(size 1.27 1.27)
-			)
-			(justify left)
-		)
-	)
 	(hierarchical_label "D14"
 		(shape tri_state)
@@
 		)
 	)
+	(hierarchical_label "JCC2"
+		(shape output)
+		(at 120.65 30.48 90)
+		(effects
+			(font
+				(size 1.27 1.27)
+			)
+			(justify left)
+		)
+	)
 	(hierarchical_label "D3"
 		(shape tri_state)
@@
 		(effects
 			(font
-				(size 1.27 1.27)
-			)
-			(justify left)
-		)
-	)
-	(hierarchical_label "RES2"
-		(shape output)
-		(at 120.65 30.48 90)
-		(effects
-			(font
