File: fr.kicad_sch (KiCad schematic)
At the start: 16 parts, among them J29 574_CP, Q28 BC557, Q29 BC547, Q30 BC547, U93 74HC245, U96 74HC574_w_Pwr, U99 74LS157

Commit message: feat: added IR into motherboard
Connections:
- net FR_IN renamed FR_IN#
Changed lines of the file:
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@@
 		)
 	)
-	(hierarchical_label "FR_IN"
+	(hierarchical_label "FR_IN#"
 		(shape input)
 		(at 233.68 163.83 270)

Commit message: WIP: created but not finished cl
Connections:
- net FR_OV_OUT: now reaches U93.11 (B7), U96.12 (Q7)
- net FR_S_OUT: now reaches U93.13 (B5), U96.14 (Q5)
- net FR_Z_OUT: now reaches U93.14 (B4), U96.15 (Q4)
- net FR_CARRY_OUT renamed FR_C_OUT
Changed lines of the file:
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@@
+	)
+	(junction
+		(at 77.47 38.1)
+		(diameter 0)
+		(color 0 0 0 0)
 	)
 	(junction
@@
 		(color 0 0 0 0)
 	)
+	(junction
+		(at 85.09 34.29)
+		(diameter 0)
+		(color 0 0 0 0)
+	)
+	(junction
+		(at 80.01 36.83)
+		(diameter 0)
+		(color 0 0 0 0)
+	)
 	(wire
 		(pts
@@
 	(wire
 		(pts
+			(xy 77.47 24.13) (xy 77.47 38.1)
+		)
+		(stroke
+			(width 0)
+			(type default)
+		)
+	)
+	(wire
+		(pts
 			(xy 138.43 72.39) (xy 124.46 72.39)
 		)
@@
 	(wire
 		(pts
+			(xy 80.01 24.13) (xy 80.01 36.83)
+		)
+		(stroke
+			(width 0)
+			(type default)
+		)
+	)
+	(wire
+		(pts
 			(xy 273.05 107.95) (xy 279.4 107.95)
 		)
@@
 		(pts
 			(xy 114.3 236.22) (xy 82.55 236.22)
+		)
+		(stroke
+			(width 0)
+			(type default)
+		)
+	)
+	(wire
+		(pts
+			(xy 85.09 24.13) (xy 85.09 34.29)
 		)
 		(stroke
@@
 		)
 	)
+	(hierarchical_label "FR_Z_OUT"
+		(shape output)
+		(at 77.47 24.13 90)
+		(effects
+			(font
+				(size 1.27 1.27)
+			)
+			(justify left)
+		)
+	)
 	(hierarchical_label "FR_DATA_C"
 		(shape tri_state)
@@
 		)
 	)
+	(hierarchical_label "FR_S_OUT"
+		(shape output)
+		(at 80.01 24.13 90)
+		(effects
+			(font
+				(size 1.27 1.27)
+			)
+			(justify left)
+		)
+	)
 	(hierarchical_label "FR_IN#"
 		(shape input)
@@
 		)
 	)
+	(hierarchical_label "FR_OV_OUT"
+		(shape output)
+		(at 85.09 24.13 90)
+		(effects
+			(font
+				(size 1.27 1.27)
+			)
+			(justify left)
+		)
+	)
 	(hierarchical_label "GND"
 		(shape input)
@@
 		)
 	)
-	(hierarchical_label "FR_CARRY_OUT"
-		(shape input)
-		(at 82.55 24.13 180)
-		(effects
-			(font
-				(size 1.27 1.27)
-			)
-			(justify right)
-		)
-	)
+	(hierarchical_label "FR_C_OUT"
+		(shape output)
+		(at 82.55 24.13 90)
+		(effects
+			(font
+				(size 1.27 1.27)
+			)
+			(justify left)
+		)
+	)
