File: cl.kicad_sch (KiCad schematic)
At the start: 2 parts, among them U142 74LS151

Commit message: feat: finished cl
Parts:
- added C151: 100nF, Capacitor_THT:C_Disc_D3.0mm_W1.6mm_P2.50mm, symbol Device:C
- added U141: 74HC04, Package_CSP:Xilinx_CSG48_7.0x7.0mm_Layout7x7_P0.8mm, symbol 74xx:74HC04
Connections:
- net at U142.1 (I3): now also U141.4
- net at U142.12 (I7): now also U141.8
- net FLAG_OV: now reaches U142.13 (I6)
- net FLAG_OV: now also U141.9
- net at U142.14 (I5): now also U141.6
- net FLAG_S: now reaches U142.15 (I4)
- net FLAG_S: now also U141.5
- net Vcc: now reaches C150.1, U142.16 (VCC)
- net Vcc: now also C151.1, U141.14 (VCC)
- net FLAG_C: now reaches U142.2 (I2)
- net FLAG_C: now also U141.3
- net at U142.3 (I1): now also U141.2
- net FLAG_Z: now reaches U142.4 (I0)
- net FLAG_Z: now also U141.1
- net JUMP_TAKEN: now reaches U142.5 (Z)
- net GND: now reaches C150.2, U142.7 (~{E}), U142.8 (GND)
- net GND: now also C151.2, U141.7 (GND)
