File: alu.kicad_sch (KiCad schematic)
At the start: 92 parts, among them U34 74LS153, U35 74HC138, U37 74HC04, U38 74HC04, U39 74HC04, U40 74HC86, U41 74HC86, U42 74HC86, U51 74HC86, U52 74HC86, U53 74HC86, U54 74HC86, U57 74HC86, U60 74HC86, U61 74LS08, U62 74LS08, U63 74LS08, U64 74LS08, U65 74LS32, U66 74LS32, U67 74LS32, U68 74LS32, U69 74HC245, U70 74HC245, U71 74HC245, U72 74HC245, U73 74HC245, U74 74HC245, U75 74LS283, U76 74LS283, U77 74LS283, U78 74LS283, U79 74HC245, U80 74HC245, U81 74HC245, U82 74HC245, U83 74HC245, U84 74HC245, U85 74HC245, U86 74HC245, U87 74LS157, U88 74LS08, U89 74LS32, U90 74LS32, U91 74LS32, U92 74LS32

Commit message: feat: connected all control signals to cu
Changed lines of the file:
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@@
 		)
 	)
-	(hierarchical_label "ALU_A_IN"
+	(hierarchical_label "#ALU_A_IN"
 		(shape input)
 		(at 500.38 515.62 270)
@@
 		)
 	)
-	(hierarchical_label "ALU_B_IN"
+	(hierarchical_label "#ALU_B_IN"
 		(shape input)
 		(at 502.92 515.62 270)
