File: HOMER1.kicad_sch (KiCad schematic)
At the start: 12 parts, among them U1 74HC138, U130 74HC138, U131 74HC138, U132 74HC138, U2 74HC138, U3 74HC138

Commit message: feat: added IR into motherboard
Parts:
- added C142, C143, C144: 100nF, Capacitor_THT:C_Disc_D3.0mm_W1.6mm_P2.50mm, symbol Device:C
- added U137: 74HC138, symbol 74xx:74HC138
- added U138, U139: 74HC00, symbol 74xx:74HC00
Connections:
- net Flags Register/FR_DATA_OUT: now also U3.9 (~{Y6})
- net GPR/GPR_DATA_OUT#: now also U139.11; no longer U1.15 (~{Y0})
- net GPR1/GPR_DATA_OUT#: now also U139.8; no longer U1.14 (~{Y1})
- net GPR2/GPR_DATA_OUT#: now also U139.6; no longer U1.13 (~{Y2})
- net GPR3/GPR_DATA_OUT#: now also U139.3; no longer U1.12 (~{Y3})
- net GPR4/GPR_DATA_OUT#: now also U138.11; no longer U1.11 (~{Y4})
- net GPR5/GPR_DATA_OUT#: now also U138.8; no longer U1.10 (~{Y5})
- net GPR6/GPR_DATA_OUT#: now also U138.6; no longer U1.9 (~{Y6})
- net GPR7/GPR_DATA_OUT#: now also U138.3; no longer U1.7 (~{Y7})
- net Heap Pointer/HP_ADDR_OUT#: now also U131.14 (~{Y1})
- net Heap Pointer/HP_COUNT_EN#: now also U132.14 (~{Y1})
- net Heap Pointer/HP_DATA_IN#: now also U130.14 (~{Y1})
- net Heap Pointer/HP_DATA_OUT#: now also U3.14 (~{Y1})
- net Memory Controller/BANK_DATA_IN#: now also U130.12 (~{Y3})
- net Memory Controller/BANK_DATA_OUT#: now also U3.12 (~{Y3})
- net Memory Controller/MEMORY_DATA_IN#: now also U130.11 (~{Y4})
- net Memory Controller/MEMORY_DATA_OUT#: now also U3.11 (~{Y4})
- net Memory Data Register/MDR_DATA_IN#: now also U130.10 (~{Y5})
- net Memory Data Register/MDR_DATA_OUT#: now also U3.10 (~{Y5})
- net Program Counter/PC_ADDR_OUT#: now also U131.15 (~{Y0})
- net Program Counter/PC_COUNT_EN#: now also U132.15 (~{Y0})
- net Program Counter/PC_DATA_IN#: now also U130.15 (~{Y0})
- net Program Counter/PC_DATA_OUT#: now also U3.15 (~{Y0})
- net Stack Pointer/HP_ADDR_OUT#: now also U131.13 (~{Y2})
- net Stack Pointer/HP_COUNT_EN#: now also U132.13 (~{Y2})
- net Stack Pointer/HP_DATA_IN#: now also U130.13 (~{Y2})
- net Stack Pointer/HP_DATA_OUT#: now also U3.13 (~{Y2})
- net at C123.1, C124.1, U1.16 (VCC)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: now also C142.1, C143.1, C144.1, U137.16 (VCC), U138.14 (VCC), U139.14 (VCC)
- net at U2.4 (~{E0}): now also C123.2, C124.2, U1.4 (~{E0}), U1.5 (~{E1}), U1.8 (GND), U2.5 (~{E1}), U2.8 (GND), C142.2, C143.2, C144.2, U137.4 (~{E0}), U137.5 (~{E1}), U137.8 (GND), U138.7 (GND), U139.7 (GND)
- net at C133.2, C134.2, C135.2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: now also U131.3 (A2), U132.3 (A2); no longer U3.3 (A2)
- net IR/IR_DATA_IN#: now reaches U130.9 (~{Y6})
- new net: U1.9 (~{Y6}), U138.4
- new net: U137.9 (~{Y6}), U138.5
- new net: U1.15 (~{Y0}), U139.12
- new net: U137.15 (~{Y0}), U139.13
- new net: U1.13 (~{Y2}), U139.4
- new net: U137.13 (~{Y2}), U139.5
- new net: U137.14 (~{Y1}), U139.10
- new net: U1.14 (~{Y1}), U139.9
- new net: U1.7 (~{Y7}), U138.1
- new net: U137.7 (~{Y7}), U138.2
- new net: U1.11 (~{Y4}), U138.12
- new net: U137.11 (~{Y4}), U138.13
- new net: U1.12 (~{Y3}), U139.1
- new net: U137.12 (~{Y3}), U139.2
- new net: U137.10 (~{Y5}), U138.10
- new net: U1.10 (~{Y5}), U138.9
Other:
- added sheet IR (IR.kicad_sch)
- sheet Flags Register ports: added FR_IN#; removed FR_IN
- sheet Memory Adress Register ports: added MAR_GATE[0->DATA;1->ADDR]; removed MAR_ADDR_GATE#, MAR_DATA_GATE#
- note added: "#_ADDR_OUT"
- note added: "#_DATA_IN"
- note added: "#_DATA_OUT"
- note added: "#_count_en"
- note added: "Count_Direction"
- note added: "MAR_SIGNALS"
- moved on the sheet: C133, C134, C135, C136, U130, U131, U132, U3

Commit message: WIP: created but not finished cl
Connections:
- net IR/RS20: now also U1.1 (A0)
- net IR/RS21: now also U1.2 (A1)
- net IR/RS22: now also U1.3 (A2)
- net IR/RS/RD0: now also U137.1 (A0), U2.1 (A0)
- net IR/RS/RD1: now also U137.2 (A1), U2.2 (A1)
- net IR/RS/RD2: now also U137.3 (A2), U2.3 (A2)
Other:
- added sheet Control Logic (cl.kicad_sch)
- added sheet Control Unit (cu.kicad_sch)
- sheet Flags Register ports: added FR_C_OUT, FR_OV_OUT, FR_S_OUT, FR_Z_OUT; removed FR_CARRY_OUT
- sheet IR ports: added BIT0, JCC0, JCC1, JCC2; removed 0, RES0, RES1, RES2
- note added: "CARRY_FLAG"
- note added: "FR_INSTANT_FLAGS"
- note added: "OVERFLOW_FLAG"
- note added: "REG_DST_IN"
- note added: "REG_SRC1_OUT"
- note added: "REG_SRC2_OUT"
- note added: "SIGN_FLAG"
- note added: "ZERO_FLAG"

Commit message: feat: finished cl
Other:
- sheet Control Logic ports: added FLAG_C, FLAG_OV, FLAG_S, FLAG_Z, GND, JUMP_TAKEN, Vcc; removed none
Changed lines of the file:
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@@
 	)
 	(junction
+		(at 384.81 694.69)
+		(diameter 0)
+		(color 0 0 0 0)
+	)
+	(junction
 		(at 67.31 194.31)
 		(diameter 0)
@@
 	)
 	(junction
+		(at 387.35 693.42)
+		(diameter 0)
+		(color 0 0 0 0)
+	)
+	(junction
 		(at 397.51 292.1)
 		(diameter 0)
@@
 	(wire
 		(pts
+			(xy 384.81 694.69) (xy 384.81 698.5)
+		)
+		(stroke
+			(width 0)
+			(type default)
+		)
+	)
+	(wire
+		(pts
 			(xy 420.37 269.24) (xy 420.37 276.86)
 		)
@@
 	(wire
 		(pts
-			(xy 441.96 656.59) (xy 361.95 656.59)
+			(xy 444.5 656.59) (xy 361.95 656.59)
 		)
 		(stroke
@@
 	(wire
 		(pts
-			(xy 444.5 655.32) (xy 444.5 721.36)
+			(xy 447.04 655.32) (xy 447.04 736.6)
 		)
 		(stroke
@@
 	(wire
 		(pts
-			(xy 466.09 745.49) (xy 669.29 745.49)
-		)
-		(stroke
-			(width 0)
-			(type default)
-		)
-	)
-	(wire
-		(pts
 			(xy 591.82 627.38) (xy 626.11 627.38)
 		)
@@
 	(wire
 		(pts
-			(xy 439.42 657.86) (xy 359.41 657.86)
+			(xy 441.96 657.86) (xy 359.41 657.86)
 		)
 		(stroke
@@
 	(wire
 		(pts
-			(xy 384.81 615.95) (xy 384.81 698.5)
+			(xy 384.81 615.95) (xy 384.81 694.69)
 		)
 		(stroke
@@
 	(wire
 		(pts
-			(xy 441.96 656.59) (xy 441.96 721.36)
+			(xy 444.5 656.59) (xy 444.5 736.6)
 		)
 		(stroke
@@
 	(wire
 		(pts
-			(xy 521.97 681.99) (xy 560.07 681.99)
+			(xy 457.2 745.49) (xy 669.29 745.49)
 		)
 		(stroke
@@
 	(wire
 		(pts
-			(xy 384.81 554.99) (xy 436.88 554.99)
+			(xy 521.97 681.99) (xy 560.07 681.99)
 		)
 		(stroke
@@
 	(wire
 		(pts
-			(xy 466.09 750.57) (xy 674.37 750.57)
+			(xy 384.81 554.99) (xy 436.88 554.99)
 		)
 		(stroke
@@
 	(wire
 		(pts
+			(xy 435.61 736.6) (xy 435.61 693.42)
+		)
+		(stroke
+			(width 0)
+			(type default)
+		)
+	)
+	(wire
+		(pts
 			(xy 433.07 29.21) (xy 447.04 29.21)
 		)
@@
 	(wire
 		(pts
+			(xy 387.35 693.42) (xy 435.61 693.42)
+		)
+		(stroke
+			(width 0)
+			(type default)
+		)
+	)
+	(wire
+		(pts
 			(xy 524.51 633.73) (xy 524.51 257.81)
 		)
@@
 	(wire
 		(pts
+			(xy 457.2 750.57) (xy 674.37 750.57)
+		)
+		(stroke
+			(width 0)
+			(type default)
+		)
+	)
+	(wire
+		(pts
 			(xy 361.95 656.59) (xy 361.95 612.14)
 		)
@@
 	(wire
 		(pts
+			(xy 457.2 748.03) (xy 671.83 748.03)
+		)
+		(stroke
+			(width 0)
+			(type default)
+		)
+	)
+	(wire
+		(pts
 			(xy 425.45 515.62) (xy 425.45 568.96)
 		)
@@
 	(wire
 		(pts
-			(xy 466.09 742.95) (xy 666.75 742.95)
-		)
-		(stroke
-			(width 0)
-			(type default)
-		)
-	)
-	(wire
-		(pts
 			(xy 430.53 259.08) (xy 430.53 266.7)
 		)
@@
 	(wire
 		(pts
-			(xy 444.5 655.32) (xy 364.49 655.32)
+			(xy 447.04 655.32) (xy 364.49 655.32)
 		)
 		(stroke
@@
 	(wire
 		(pts
+			(xy 433.07 694.69) (xy 384.81 694.69)
+		)
+		(stroke
+			(width 0)
+			(type default)
+		)
+	)
+	(wire
+		(pts
 			(xy 379.73 63.5) (xy 387.35 63.5)
 		)
@@
 	(wire
 		(pts
+			(xy 457.2 742.95) (xy 666.75 742.95)
+		)
+		(stroke
+			(width 0)
+			(type default)
+		)
+	)
+	(wire
+		(pts
 			(xy 364.49 250.19) (xy 293.37 250.19)
 		)
@@
 	(wire
 		(pts
+			(xy 387.35 693.42) (xy 387.35 698.5)
+		)
+		(stroke
+			(width 0)
+			(type default)
+		)
+	)
+	(wire
+		(pts
 			(xy 389.89 236.22) (xy 389.89 245.11)
 		)
@@
 	(wire
 		(pts
-			(xy 387.35 613.41) (xy 387.35 698.5)
+			(xy 387.35 613.41) (xy 387.35 693.42)
 		)
 		(stroke
@@
 	(wire
 		(pts
-			(xy 439.42 657.86) (xy 439.42 721.36)
+			(xy 441.96 657.86) (xy 441.96 736.6)
 		)
 		(stroke
@@
 	(wire
 		(pts
-			(xy 466.09 748.03) (xy 671.83 748.03)
+			(xy 422.91 758.19) (xy 430.53 758.19)
 		)
 		(stroke
@@
 	(wire
 		(pts
+			(xy 433.07 736.6) (xy 433.07 694.69)
+		)
+		(stroke
+			(width 0)
+			(type default)
+		)
+	)
+	(wire
+		(pts
 			(xy 378.46 207.01) (xy 420.37 207.01)
 		)
@@
 		)
 		(pin "INTERRUPT_ACTIVE" input
-			(at 278.13 786.13 180)
+			(at 278.13 784.86 180)
 			(effects
 				(font
@@
 		)
 		(pin "JUMP_TAKEN" input
-			(at 278.13 783.59 180)
+			(at 422.91 758.19 0)
 			(effects
 				(font
 					(size 1.27 1.27)
 				)
-				(justify left)
+				(justify right)
 			)
 		)
@@
 	)
 	(sheet
-		(at 434.34 721.36)
-		(size 22.86 49.53)
+		(at 430.53 736.6)
+		(size 26.67 25.4)
 		(exclude_from_sim no)
 		(in_bom yes)
@@
 		)
 		(property "Sheetname" "Control Logic"
-			(at 433.578 734.822 90)
+			(at 429.768 750.062 90)
 			(show_name no)
 			(do_not_autoplace no)
@@
 		)
 		(property "Sheetfile" "cl.kicad_sch"
-			(at 434.34 771.4746 0)
+			(at 430.784 763.778 0)
 			(show_name no)
 			(do_not_autoplace no)
@@
 		)
 		(pin "JCC0" input
-			(at 444.5 721.36 90)
+			(at 447.04 736.6 90)
 			(effects
 				(font
@@
 		)
 		(pin "JCC1" input
-			(at 441.96 721.36 90)
+			(at 444.5 736.6 90)
 			(effects
 				(font
@@
 		)
 		(pin "JCC2" input
-			(at 439.42 721.36 90)
+			(at 441.96 736.6 90)
+			(effects
+				(font
+					(size 1.27 1.27)
+				)
+				(justify right)
+			)
+		)
+		(pin "FLAG_C" input
+			(at 457.2 750.57 0)
+			(effects
+				(font
+					(size 1.27 1.27)
+				)
+				(justify right)
+			)
+		)
+		(pin "FLAG_OV" input
+			(at 457.2 745.49 0)
+			(effects
+				(font
+					(size 1.27 1.27)
+				)
+				(justify right)
+			)
+		)
+		(pin "FLAG_S" input
+			(at 457.2 742.95 0)
+			(effects
+				(font
+					(size 1.27 1.27)
+				)
+				(justify right)
+			)
+		)
+		(pin "FLAG_Z" input
+			(at 457.2 748.03 0)
+			(effects
+				(font
+					(size 1.27 1.27)
+				)
+				(justify right)
+			)
+		)
+		(pin "JUMP_TAKEN" output
+			(at 430.53 758.19 180)
+			(effects
+				(font
+					(size 1.27 1.27)
+				)
+				(justify left)
+			)
+		)
+		(pin "GND" input
+			(at 435.61 736.6 90)
+			(effects
+				(font
+					(size 1.27 1.27)
+				)
+				(justify right)
+			)
+		)
+		(pin "Vcc" input
+			(at 433.07 736.6 90)
 			(effects
 				(font

Commit message: feat: connected all control signals to cu
Parts:
- added C149, C160: 100nF, Capacitor_THT:C_Disc_D3.0mm_W1.6mm_P2.50mm, symbol Device:C
- added EXDP0, EXDP1, EXDP2, EXDP3, EXDP4, EXDP5, EXDP6, EXDP7: Conn_01x17_Socket, symbol Connector:Conn_01x17_Socket
- added J47, J48, J49, J50, J51, J52, J53, J54: EXDP1, symbol Connector:Conn_01x20_Socket
- added U148, U150: 74HC138, symbol 74xx:74HC138
Connections:
- net +5V: now also J47.1 (Pin_1), J48.1 (Pin_1), J49.1 (Pin_1), J50.1 (Pin_1), J51.1 (Pin_1), J52.1 (Pin_1), J53.1 (Pin_1), J54.1 (Pin_1)
- net Arthmetic Logic Unit/CLK: now also J47.3 (Pin_3), J48.3 (Pin_3), J49.3 (Pin_3), J50.3 (Pin_3), J51.3 (Pin_3), J52.3 (Pin_3), J53.3 (Pin_3), J54.3 (Pin_3)
- net Arthmetic Logic Unit/D0: now also J47.20 (Pin_20), J48.20 (Pin_20), J49.20 (Pin_20), J50.20 (Pin_20), J51.20 (Pin_20), J52.20 (Pin_20), J53.20 (Pin_20), J54.20 (Pin_20)
- net Arthmetic Logic Unit/D1: now also J47.19 (Pin_19), J48.19 (Pin_19), J49.19 (Pin_19), J50.19 (Pin_19), J51.19 (Pin_19), J52.19 (Pin_19), J53.19 (Pin_19), J54.19 (Pin_19)
- net Arthmetic Logic Unit/D10: now also J47.10 (Pin_10), J48.10 (Pin_10), J49.10 (Pin_10), J50.10 (Pin_10), J51.10 (Pin_10), J52.10 (Pin_10), J53.10 (Pin_10), J54.10 (Pin_10)
- net Arthmetic Logic Unit/D11: now also J47.9 (Pin_9), J48.9 (Pin_9), J49.9 (Pin_9), J50.9 (Pin_9), J51.9 (Pin_9), J52.9 (Pin_9), J53.9 (Pin_9), J54.9 (Pin_9)
- net Arthmetic Logic Unit/D12: now also J47.8 (Pin_8), J48.8 (Pin_8), J49.8 (Pin_8), J50.8 (Pin_8), J51.8 (Pin_8), J52.8 (Pin_8), J53.8 (Pin_8), J54.8 (Pin_8)
- net Arthmetic Logic Unit/D13: now also J47.7 (Pin_7), J48.7 (Pin_7), J49.7 (Pin_7), J50.7 (Pin_7), J51.7 (Pin_7), J52.7 (Pin_7), J53.7 (Pin_7), J54.7 (Pin_7)
- net Arthmetic Logic Unit/D14: now also J47.6 (Pin_6), J48.6 (Pin_6), J49.6 (Pin_6), J50.6 (Pin_6), J51.6 (Pin_6), J52.6 (Pin_6), J53.6 (Pin_6), J54.6 (Pin_6)
- net Arthmetic Logic Unit/D15: now also J47.5 (Pin_5), J48.5 (Pin_5), J49.5 (Pin_5), J50.5 (Pin_5), J51.5 (Pin_5), J52.5 (Pin_5), J53.5 (Pin_5), J54.5 (Pin_5)
- net Arthmetic Logic Unit/D2: now also J47.18 (Pin_18), J48.18 (Pin_18), J49.18 (Pin_18), J50.18 (Pin_18), J51.18 (Pin_18), J52.18 (Pin_18), J53.18 (Pin_18), J54.18 (Pin_18)
- net Arthmetic Logic Unit/D3: now also J47.17 (Pin_17), J48.17 (Pin_17), J49.17 (Pin_17), J50.17 (Pin_17), J51.17 (Pin_17), J52.17 (Pin_17), J53.17 (Pin_17), J54.17 (Pin_17)
- net Arthmetic Logic Unit/D4: now also J47.16 (Pin_16), J48.16 (Pin_16), J49.16 (Pin_16), J50.16 (Pin_16), J51.16 (Pin_16), J52.16 (Pin_16), J53.16 (Pin_16), J54.16 (Pin_16)
- net Arthmetic Logic Unit/D5: now also J47.15 (Pin_15), J48.15 (Pin_15), J49.15 (Pin_15), J50.15 (Pin_15), J51.15 (Pin_15), J52.15 (Pin_15), J53.15 (Pin_15), J54.15 (Pin_15)
- net Arthmetic Logic Unit/D6: now also J47.14 (Pin_14), J48.14 (Pin_14), J49.14 (Pin_14), J50.14 (Pin_14), J51.14 (Pin_14), J52.14 (Pin_14), J53.14 (Pin_14), J54.14 (Pin_14)
- net Arthmetic Logic Unit/D7: now also J47.13 (Pin_13), J48.13 (Pin_13), J49.13 (Pin_13), J50.13 (Pin_13), J51.13 (Pin_13), J52.13 (Pin_13), J53.13 (Pin_13), J54.13 (Pin_13)
- net Arthmetic Logic Unit/D8: now also J47.12 (Pin_12), J48.12 (Pin_12), J49.12 (Pin_12), J50.12 (Pin_12), J51.12 (Pin_12), J52.12 (Pin_12), J53.12 (Pin_12), J54.12 (Pin_12)
- net Arthmetic Logic Unit/D9: now also J47.11 (Pin_11), J48.11 (Pin_11), J49.11 (Pin_11), J50.11 (Pin_11), J51.11 (Pin_11), J52.11 (Pin_11), J53.11 (Pin_11), J54.11 (Pin_11)
- net GND: now also J47.2 (Pin_2), J48.2 (Pin_2), J49.2 (Pin_2), J50.2 (Pin_2), J51.2 (Pin_2), J52.2 (Pin_2), J53.2 (Pin_2), J54.2 (Pin_2)
- net IR/IR_DATA_OUT#: now also U150.14 (~{Y1})
- net Memory Adress Register/M0: now also EXDP0.5 (Pin_5), EXDP1.5 (Pin_5), EXDP2.5 (Pin_5), EXDP3.5 (Pin_5), EXDP4.5 (Pin_5), EXDP5.5 (Pin_5), EXDP6.5 (Pin_5), EXDP7.5 (Pin_5)
- net Memory Adress Register/M1: now also EXDP0.6 (Pin_6), EXDP1.6 (Pin_6), EXDP2.6 (Pin_6), EXDP3.6 (Pin_6), EXDP4.6 (Pin_6), EXDP5.6 (Pin_6), EXDP6.6 (Pin_6), EXDP7.6 (Pin_6)
- net Memory Adress Register/M10: now also EXDP0.15 (Pin_15), EXDP1.15 (Pin_15), EXDP2.15 (Pin_15), EXDP3.15 (Pin_15), EXDP4.15 (Pin_15), EXDP5.15 (Pin_15), EXDP6.15 (Pin_15), EXDP7.15 (Pin_15)
- net Memory Adress Register/M11: now also EXDP0.16 (Pin_16), EXDP1.16 (Pin_16), EXDP2.16 (Pin_16), EXDP3.16 (Pin_16), EXDP4.16 (Pin_16), EXDP5.16 (Pin_16), EXDP6.16 (Pin_16), EXDP7.16 (Pin_16)
- net Memory Adress Register/M12: now also EXDP0.17 (Pin_17), EXDP1.17 (Pin_17), EXDP2.17 (Pin_17), EXDP3.17 (Pin_17), EXDP4.17 (Pin_17), EXDP5.17 (Pin_17), EXDP6.17 (Pin_17), EXDP7.17 (Pin_17)
- net Memory Adress Register/M13: now also U148.1 (A0)
- net Memory Adress Register/M14: now also U148.2 (A1)
- net Memory Adress Register/M15: now also U148.3 (A2)
- net Memory Adress Register/M2: now also EXDP0.7 (Pin_7), EXDP1.7 (Pin_7), EXDP2.7 (Pin_7), EXDP3.7 (Pin_7), EXDP4.7 (Pin_7), EXDP5.7 (Pin_7), EXDP6.7 (Pin_7), EXDP7.7 (Pin_7)
- net Memory Adress Register/M3: now also EXDP0.8 (Pin_8), EXDP1.8 (Pin_8), EXDP2.8 (Pin_8), EXDP3.8 (Pin_8), EXDP4.8 (Pin_8), EXDP5.8 (Pin_8), EXDP6.8 (Pin_8), EXDP7.8 (Pin_8)
- net Memory Adress Register/M4: now also EXDP0.9 (Pin_9), EXDP1.9 (Pin_9), EXDP2.9 (Pin_9), EXDP3.9 (Pin_9), EXDP4.9 (Pin_9), EXDP5.9 (Pin_9), EXDP6.9 (Pin_9), EXDP7.9 (Pin_9)
- net Memory Adress Register/M5: now also EXDP0.10 (Pin_10), EXDP1.10 (Pin_10), EXDP2.10 (Pin_10), EXDP3.10 (Pin_10), EXDP4.10 (Pin_10), EXDP5.10 (Pin_10), EXDP6.10 (Pin_10), EXDP7.10 (Pin_10)
- net Memory Adress Register/M6: now also EXDP0.11 (Pin_11), EXDP1.11 (Pin_11), EXDP2.11 (Pin_11), EXDP3.11 (Pin_11), EXDP4.11 (Pin_11), EXDP5.11 (Pin_11), EXDP6.11 (Pin_11), EXDP7.11 (Pin_11)
- net Memory Adress Register/M7: now also EXDP0.12 (Pin_12), EXDP1.12 (Pin_12), EXDP2.12 (Pin_12), EXDP3.12 (Pin_12), EXDP4.12 (Pin_12), EXDP5.12 (Pin_12), EXDP6.12 (Pin_12), EXDP7.12 (Pin_12)
- net Memory Adress Register/M8: now also EXDP0.13 (Pin_13), EXDP1.13 (Pin_13), EXDP2.13 (Pin_13), EXDP3.13 (Pin_13), EXDP4.13 (Pin_13), EXDP5.13 (Pin_13), EXDP6.13 (Pin_13), EXDP7.13 (Pin_13)
- net Memory Adress Register/M9: now also EXDP0.14 (Pin_14), EXDP1.14 (Pin_14), EXDP2.14 (Pin_14), EXDP3.14 (Pin_14), EXDP4.14 (Pin_14), EXDP5.14 (Pin_14), EXDP6.14 (Pin_14), EXDP7.14 (Pin_14)
- net Memory Controller/MEMORY_DATA_IN#: now also EXDP0.3 (Pin_3), EXDP1.3 (Pin_3), EXDP2.3 (Pin_3), EXDP3.3 (Pin_3), EXDP4.3 (Pin_3), EXDP5.3 (Pin_3), EXDP6.3 (Pin_3), EXDP7.3 (Pin_3)
- net Memory Controller/MEMORY_DATA_OUT#: now also EXDP0.4 (Pin_4), EXDP1.4 (Pin_4), EXDP2.4 (Pin_4), EXDP3.4 (Pin_4), EXDP4.4 (Pin_4), EXDP5.4 (Pin_4), EXDP6.4 (Pin_4), EXDP7.4 (Pin_4)
- net Memory Controller/MMIO_CS#: now also U148.5 (~{E1})
- net at C123.1, C124.1, C142.1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: now also U1.6 (E2), U137.6 (E2), U2.6 (E2)
- net at C123.2, C124.2, C142.2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: no longer U1.4 (~{E0}), U137.4 (~{E0}), U2.4 (~{E0})
- net Control Unit/DATA_IN0: now reaches U130.1 (A0)
- net at C133.1, C134.1, C135.1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: now also U130.6 (E2), U131.6 (E2), U132.6 (E2), U3.6 (E2), C160.1, U150.16 (VCC)
- net Control Unit/DATA_IN1: now reaches U130.2 (A1)
- net Control Unit/DATA_IN2: now reaches U130.3 (A2)
- net Control Unit/#DATA_IN_EN: now reaches U130.4 (~{E0})
- net at U130.5 (~{E1}): now also C133.2, C134.2, C135.2, C136.2, U130.8 (GND), U131.3 (A2), U131.4 (~{E0}), U131.5 (~{E1}), U131.8 (GND), U132.3 (A2), U132.4 (~{E0}), U132.5 (~{E1}), U132.8 (GND), U3.5 (~{E1}), U3.8 (GND), C160.2, U150.3 (A2), U150.4 (~{E0}), U150.5 (~{E1}), U150.8 (GND)
- net at U130.7 (~{Y7}): now also U2.4 (~{E0})
- net Control Unit/COUNT_EN0: now reaches U132.1 (A0)
- net Control Unit/COUNT_EN1: now reaches U132.2 (A1)
- net Control Unit/DATA_OUT2_0: now reaches U3.1 (A0)
- net Control Unit/DATA_OUT2_1: now reaches U3.2 (A1)
- net Control Unit/DATA_OUT2_2: now reaches U3.3 (A2)
- net Control Unit/DATA_OUT_SRC: now reaches U3.4 (~{E0})
- net Control Unit/DATA_OUT_SRC: now also U150.6 (E2)
- net Control Unit/ADDR_OUT0: now reaches U131.1 (A0)
- net Control Unit/ADDR_OUT1: now reaches U131.2 (A1)
- new net: EXDP3.1 (Pin_1), U148.12 (~{Y3})
- new net: EXDP5.1 (Pin_1), U148.10 (~{Y5})
- new net: EXDP4.1 (Pin_1), U148.11 (~{Y4})
- new net: EXDP2.1 (Pin_1), U148.13 (~{Y2})
- new net: EXDP1.1 (Pin_1), U148.14 (~{Y1})
- new net: EXDP0.1 (Pin_1), U148.15 (~{Y0})
- new net: C149.1, U148.16 (VCC), U148.6 (E2)
- new net: C149.2, U148.4 (~{E0}), U148.8 (GND)
- new net: EXDP7.1 (Pin_1), U148.7 (~{Y7})
- new net: EXDP6.1 (Pin_1), U148.9 (~{Y6})
- new net: J47.4 (Pin_4), J48.4 (Pin_4), J49.4 (Pin_4), J50.4 (Pin_4), J51.4 (Pin_4), J52.4 (Pin_4), J53.4 (Pin_4), J54.4 (Pin_4)
- new net: U137.4 (~{E0}), U150.12 (~{Y3})
- new net: U1.4 (~{E0}), U150.13 (~{Y2})
- new net Control Unit/DATA_OUT1_0: U150.1 (A0)
- new net Control Unit/DATA_OUT1_1: U150.2 (A1)
- new net Interrput Controller/#IC_DATA_OUT: U150.15 (~{Y0})
- new net Interrput Controller/IRQ_IN0: EXDP0.2 (Pin_2)
- new net Interrput Controller/IRQ_IN1: EXDP1.2 (Pin_2)
- new net Interrput Controller/IRQ_IN2: EXDP2.2 (Pin_2)
- new net Interrput Controller/IRQ_IN3: EXDP3.2 (Pin_2)
- new net Interrput Controller/IRQ_IN4: EXDP4.2 (Pin_2)
- new net Interrput Controller/IRQ_IN5: EXDP5.2 (Pin_2)
- new net Interrput Controller/IRQ_IN6: EXDP6.2 (Pin_2)
- new net Interrput Controller/IRQ_IN7: EXDP7.2 (Pin_2)
Other:
- added sheet Interrput Controller (ic.kicad_sch)
- sheet Arthmetic Logic Unit ports: added #ALU_A_IN, #ALU_B_IN; removed ALU_A_IN, ALU_B_IN
- sheet Control Unit ports: added #ALU_A_IN, #ALU_B_IN, #DATA_IN_EN, #END_INSTRUCTION, #FR_IN, #MAR_IN, ADDR_OUT0, ADDR_OUT1, ALU_CARRY_SEL0, ALU_CARRY_SEL1, ALU_INV_B, ALU_MODE0, ALU_MODE1, ALU_MODE2, COUNT_DIR, COUNT_EN0, COUNT_EN1, DATA_IN0, DATA_IN1, DATA_IN2, DATA_OUT1_0, DATA_OUT1_1, DATA_OUT2_0, DATA_OUT2_1, DATA_OUT2_2, DATA_OUT_SRC, ENTER_SUPERVISOR, FR_SRC_SEL, IRQ_CLEAR, MAR_GATE; removed SUPERVISOR_MODE
- note added: "#ALU_A_IN"
- note added: "#ALU_B_IN"
- note added: "#DATA_IN_EN <-------"
- note added: "#DATA_OUT_SRC <---------"
- note added: "#FR_IN"
- note added: "#_DATA_OUT1"
- note added: "#_DATA_OUT2"
- note added: "ALU_CARRY_SEL0"
- note added: "ALU_CARRY_SEL1"
- note added: "ALU_INV_B"
- note added: "ALU_MODE0"
- note added: "ALU_MODE1"
- note added: "ALU_MODE2"
- note added: "FR_SRC_SEL"
- note added: "IC signals"
- note added: "|-------BIT0...12-------|"
- note removed: "#_DATA_OUT"
- moved on the sheet: C123, C124, C133, C134, C135, C136, C142, C143, C144, U1, U130, U131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

Commit message: feat: created and connected all functional components
Other:
- sheet Control Unit ports: added IRQ; removed #END_INSTRUCTION, ENTER_SUPERVISOR, INTERRUPT_ACTIVE
Changed lines of the file:
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@@
 	)
 	(junction
+		(at 278.13 919.48)
+		(diameter 0)
+		(color 0 0 0 0)
+	)
+	(junction
 		(at 400.05 175.26)
 		(diameter 0)
@@
 	(wire
 		(pts
+			(xy 278.13 919.48) (xy 295.91 919.48)
+		)
+		(stroke
+			(width 0)
+			(type default)
+		)
+	)
+	(wire
+		(pts
 			(xy 410.21 287.02) (xy 410.21 347.98)
 		)
@@
 	(wire
 		(pts
+			(xy 278.13 919.48) (xy 278.13 990.6)
+		)
+		(stroke
+			(width 0)
+			(type default)
+		)
+	)
+	(wire
+		(pts
 			(xy 384.81 17.78) (xy 384.81 66.04)
 		)
@@
 	(wire
 		(pts
-			(xy 278.13 657.86) (xy 278.13 990.6)
+			(xy 278.13 657.86) (xy 278.13 919.48)
 		)
 		(stroke
@@
 			)
 		)
-		(pin "INTERRUPT_ACTIVE" input
-			(at 295.91 998.22 180)
-			(effects
-				(font
-					(size 1.27 1.27)
-				)
-				(justify left)
-			)
-		)
-		(pin "#END_INSTRUCTION" output
-			(at 295.91 988.06 180)
-			(effects
-				(font
-					(size 1.27 1.27)
-				)
-				(justify left)
-			)
-		)
-		(pin "ENTER_SUPERVISOR" input
-			(at 295.91 995.68 180)
-			(effects
-				(font
-					(size 1.27 1.27)
-				)
-				(justify left)
-			)
-		)
 		(pin "IRQ_CLEAR" output
 			(at 295.91 922.02 180)
@@
 			(effects
 				(font
+					(size 1.27 1.27)
+				)
+				(justify left)
+			)
+		)
+		(pin "IRQ" input
+			(at 295.91 919.48 180)
+			(effects
+				(font

Commit message: feat: created RESET signal
Other:
- sheet Memory Controller ports: added #RESET; removed none
- note added: "#RESET"
Changed lines of the file:
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@@
 		)
 	)
+	(text "#RESET"
+		(exclude_from_sim no)
+		(at 246.38 437.134 90)
+		(effects
+			(font
+				(size 2.54 2.54)
+			)
+		)
+	)
 	(text "#DATA_IN_EN\n<-------"
 		(exclude_from_sim no)
@@
 	(text "MAR_SIGNALS"
 		(exclude_from_sim no)
-		(at 251.714 878.332 0)
+		(at 257.556 879.602 90)
 		(effects
 			(font
@@
 		)
 	)
+	(text "#RESET"
+		(exclude_from_sim no)
+		(at 247.396 880.11 90)
+		(effects
+			(font
+				(size 2.54 2.54)
+			)
+		)
+	)
 	(text "CARRY_FLAG"
 		(exclude_from_sim no)
@@
 	)
 	(junction
+		(at 250.19 403.86)
+		(diameter 0)
+		(color 0 0 0 0)
+	)
+	(junction
 		(at 387.35 172.72)
 		(diameter 0)
@@
 	)
 	(junction
+		(at 250.19 995.68)
+		(diameter 0)
+		(color 0 0 0 0)
+	)
+	(junction
 		(at 57.15 204.47)
 		(diameter 0)
@@
 	(wire
 		(pts
+			(xy 295.91 995.68) (xy 250.19 995.68)
+		)
+		(stroke
+			(width 0)
+			(type default)
+		)
+	)
+	(wire
+		(pts
 			(xy 292.1 351.79) (xy 292.1 483.87)
 		)
@@
 	(wire
 		(pts
+			(xy 250.19 995.68) (xy 250.19 1002.03)
+		)
+		(stroke
+			(width 0)
+			(type default)
+		)
+	)
+	(wire
+		(pts
 			(xy 49.53 38.1) (xy 327.66 38.1)
 		)
@@
 	(wire
 		(pts
+			(xy 95.25 403.86) (xy 95.25 405.13)
+		)
+		(stroke
+			(width 0)
+			(type default)
+		)
+	)
+	(wire
+		(pts
 			(xy 427.99 147.32) (xy 427.99 199.39)
 		)
@@
 	(wire
 		(pts
+			(xy 250.19 403.86) (xy 95.25 403.86)
+		)
+		(stroke
+			(width 0)
+			(type default)
+		)
+	)
+	(wire
+		(pts
 			(xy 377.19 793.75) (xy 422.91 793.75)
 		)
@@
 	(wire
 		(pts
+			(xy 311.15 403.86) (xy 250.19 403.86)
+		)
+		(stroke
+			(width 0)
+			(type default)
+		)
+	)
+	(wire
+		(pts
 			(xy 36.83 288.29) (xy 311.15 288.29)
 		)
@@
 	(wire
 		(pts
+			(xy 250.19 403.86) (xy 250.19 995.68)
+		)
+		(stroke
+			(width 0)
+			(type default)
+		)
+	)
+	(wire
+		(pts
 			(xy 375.92 40.64) (xy 412.75 40.64)
 		)
@@
 			)
 		)
+		(pin "#RESET" input
+			(at 311.15 403.86 180)
+			(effects
+				(font
+					(size 1.27 1.27)
+				)
+				(justify left)
+			)
+		)
 		(instances
 			(project "HOMER1"
@@
 		)
 		(pin "#RESET" input
-			(at 422.91 998.22 0)
+			(at 295.91 995.68 180)
 			(effects
 				(font
 					(size 1.27 1.27)
 				)
-				(justify right)
+				(justify left)
 			)
 		)
