File: MC.kicad_sch (KiCad schematic)
At the start: 36 parts, among them J1_1 Conn_01x22_Socket, J1_2 Conn_01x22_Socket, J1_3 Conn_01x22_Socket, J1_4 Conn_01x22_Socket, J1_5 Conn_01x22_Socket, J1_6 Conn_01x22_Socket, J1_7 Conn_01x22_Socket, J1_8 Conn_01x22_Socket, J30 574_CP, J31 OE/A->B, Q34 BC557, Q35 BC547, Q36 BC547, U112 AS6C1008-xxP, U113 AS6C1008-xxP, U114 74HC245, U115 74HC574_w_Pwr, U118 74HC00, U119 74HC138

Commit message: feat: connected all control signals to cu
Parts:
- removed J1_1, J1_2, J1_3, J1_4, J1_5, J1_6, J1_7, J1_8: Conn_01x22_Socket, symbol Connector:Conn_01x22_Socket

Commit message: feat: created RESET signal
Parts:
- removed J30: 574_CP, Connector_PinHeader_2.54mm:PinHeader_1x02_P2.54mm_Horizontal, symbol Connector_Generic:Conn_01x02
- added C164: 100nF, Capacitor_THT:C_Disc_D3.0mm_W1.6mm_P2.50mm, symbol Device:C
- added U153: 74HC138, symbol 74xx:74HC138
Connections:
- net +5V: now also U119.6 (E2), C164.1, U153.16 (VCC)
- net GND: now also C164.2, U153.4 (~{E0}), U153.5 (~{E1}), U153.8 (GND)
- net LOW when EEPROM used: now also U119.15 (~{Y0}); no longer U119.9 (~{Y6})
- net MMIO_CS#: now also U153.7 (~{Y7}); no longer U119.7 (~{Y7})
- net at U112.2 (A16), U113.2 (A16), U114.11 (B7)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: now also U153.1 (A0)
- net at U114.12 (B6), U115.18 (Q1), U119.2 (A1): now also U153.2 (A1)
- net at U114.13 (B5), U115.17 (Q2), U119.3 (A2): now also U153.3 (A2)
- net at U114.14 (B4), U115.16 (Q3): now also U119.4 (~{E0}), U153.6 (E2); no longer U119.6 (E2)
- net at U118.10: now also Q36.3 (E), R84.1, U118.9
- net at U118.8: now also U118.13
- net at U115.11 (CP): now also U118.11
- net #RESET: now reaches U118.12
Other:
- note added: "~A OR B"
- moved on the sheet: U118A, U118B, U118C, U118D
